File: schematics/altimeter.sch (KiCad schematic (older format))
At the start: 6 parts, among them U4 TXB0106, U5 MS5611-01BA, U6 ICM-20948

Commit message: Migrate remaining symbols to local library
Parts:
- C17, C18: footprint Strix:C_0402_1005Metric_Pad0.74x0.62mm_HandSolder -> Strix:C_0402
- R7: footprint Strix:R_0402_1005Metric_Pad0.72x0.64mm_HandSolder -> Strix:R_0402
- U5: footprint Strix:LGA-8_3x5mm_P1.25mm -> Strix:MS5611-01BA
- U6: footprint Strix:InvenSense_QFN-24_3x3mm_P0.4mm -> Strix:ICM-20948
Changed lines of the file:
@@
 $Descr A4 11693 8268
 encoding utf-8
-Sheet 2 3
+Sheet 3 3
 Title "HAB Altimeter"
 Date "2021-08-31"
@@
 F 0 "C18" V 4954 3808 50  0000 L CNN
 F 1 "100n" V 5045 3808 50  0000 L CNN
-F 2 "Strix:C_0402_1005Metric_Pad0.74x0.62mm_HandSolder" H 4950 3750 50  0001 C CNN
+F 2 "Strix:C_0402" H 4950 3750 50  0001 C CNN
 F 3 "" H 4950 3750 50  0001 C CNN
 	1    4950 3750
@@
 F 0 "C17" V 4754 3808 50  0000 L CNN
 F 1 "100n" V 4845 3808 50  0000 L CNN
-F 2 "Strix:C_0402_1005Metric_Pad0.74x0.62mm_HandSolder" H 4750 3750 50  0001 C CNN
+F 2 "Strix:C_0402" H 4750 3750 50  0001 C CNN
 F 3 "" H 4750 3750 50  0001 C CNN
 	1    4750 3750
@@
 F 0 "R7" V 5404 3544 50  0000 L CNN
 F 1 "100k" V 5495 3544 50  0000 L CNN
-F 2 "Strix:R_0402_1005Metric_Pad0.72x0.64mm_HandSolder" H 5400 3500 50  0001 C CNN
+F 2 "Strix:R_0402" H 5400 3500 50  0001 C CNN
 F 3 "" H 5400 3500 50  0001 C CNN
 	1    5400 3500
@@
 F 0 "U6" H 6950 3900 50  0000 L CNN
 F 1 "ICM-20948" H 6950 3800 50  0000 L CNN
-F 2 "Strix:InvenSense_QFN-24_3x3mm_P0.4mm" H 6700 2150 50  0001 C CNN
+F 2 "Strix:ICM-20948" H 6700 2150 50  0001 C CNN
 F 3 "http://www.invensense.com/wp-content/uploads/2016/06/DS-000189-ICM-20948-v1.3.pdf" H 6700 3000 50  0001 C CNN
 	1    6700 3150
@@
 F 0 "U5" H 5200 5500 50  0000 L CNN
 F 1 "MS5611-01BA" H 5200 5400 50  0000 L CNN
-F 2 "Strix:LGA-8_3x5mm_P1.25mm" H 5000 5050 50  0001 C CNN
+F 2 "Strix:MS5611-01BA" H 5000 5050 50  0001 C CNN
 F 3 "https://www.te.com/commerce/DocumentDelivery/DDEController?Action=srchrtrv&DocNm=MS5611-01BA03&DocType=Data+Sheet&DocLang=English" H 5000 5050 50  0001 C CNN
 	1    5000 5050
