File: schematics/radio.sch (KiCad schematic (older format))
At the start: 24 parts, among them J4 BMI-S-201, U7 Si4463, U8 MAX-M8Q

Commit message: Migrate remaining symbols to local library
Parts:
- C19, C20, C21, C22, C23, C24, C25, C26, C27, C28, C29, C30: footprint Strix:C_0402_1005Metric_Pad0.74x0.62mm_HandSolder -> Strix:C_0402
- J4: footprint Strix:Laird_Technologies_BMI-S-201-F_13.66x12.70mm -> Strix:BMI-S-201; symbol Strix:RF_Shield_Two_Pieces -> Strix:BMI-S-201
- L1, L2, L3, L4, L5, L6, L7: footprint Strix:L_0402_1005Metric_Pad0.77x0.64mm_HandSolder -> Strix:L_0402
- R11, R4: footprint Strix:R_0402_1005Metric_Pad0.72x0.64mm_HandSolder -> Strix:R_0402
- U7: footprint Strix:QFN-20-1EP_4x4mm_P0.5mm_EP2.6x2.6mm_ThermalVias -> Strix:Si4463
Changed lines of the file:
@@
 F 0 "U7" H 5000 3525 50  0000 C CNN
 F 1 "Si4463" H 5000 3434 50  0000 C CNN
-F 2 "Strix:QFN-20-1EP_4x4mm_P0.5mm_EP2.6x2.6mm_ThermalVias" H 4700 1900 50  0001 L CNN
+F 2 "Strix:Si4463" H 4700 1900 50  0001 L CNN
 F 3 "" H 4600 3300 50  0001 C CNN
 F 4 "2462637" H 4700 1800 50  0001 L CNN "Farnell"
@@
 F 0 "L1" V 6904 2394 50  0000 L CNN
 F 1 "120n" V 6995 2394 50  0000 L CNN
-F 2 "Strix:L_0402_1005Metric_Pad0.77x0.64mm_HandSolder" H 6900 2350 50  0001 C CNN
+F 2 "Strix:L_0402" H 6900 2350 50  0001 C CNN
 F 3 "" H 6900 2350 50  0001 C CNN
 	1    6900 2350
@@
 F 0 "C27" H 7300 3100 50  0000 C BNN
 F 1 "1p2" H 7300 3000 50  0000 C TNN
-F 2 "Strix:C_0402_1005Metric_Pad0.74x0.62mm_HandSolder" H 7250 3050 50  0001 C CNN
+F 2 "Strix:C_0402" H 7250 3050 50  0001 C CNN
 F 3 "" H 7250 3050 50  0001 C CNN
 	1    7250 3050
@@
 F 0 "L4" H 7300 3400 50  0000 C BNN
 F 1 "24n" H 7300 3300 50  0000 C TNN
-F 2 "Strix:L_0402_1005Metric_Pad0.77x0.64mm_HandSolder" H 7250 3350 50  0001 C CNN
+F 2 "Strix:L_0402" H 7250 3350 50  0001 C CNN
 F 3 "" H 7250 3350 50  0001 C CNN
 	1    7250 3350
@@
 F 0 "C25" V 6904 3508 50  0000 L CNN
 F 1 "3p" V 6995 3508 50  0000 L CNN
-F 2 "Strix:C_0402_1005Metric_Pad0.74x0.62mm_HandSolder" H 6900 3450 50  0001 C CNN
+F 2 "Strix:C_0402" H 6900 3450 50  0001 C CNN
 F 3 "" H 6900 3450 50  0001 C CNN
 	1    6900 3450
@@
 F 0 "L2" V 6904 3194 50  0000 L CNN
 F 1 "18n" V 7000 3200 50  0000 L CNN
-F 2 "Strix:L_0402_1005Metric_Pad0.77x0.64mm_HandSolder" H 6900 3150 50  0001 C CNN
+F 2 "Strix:L_0402" H 6900 3150 50  0001 C CNN
 F 3 "" H 6900 3150 50  0001 C CNN
 	1    6900 3150
@@
 F 0 "L3" H 7300 2750 50  0000 C BNN
 F 1 "3n3" H 7300 2650 50  0000 C TNN
-F 2 "Strix:L_0402_1005Metric_Pad0.77x0.64mm_HandSolder" H 7250 2700 50  0001 C CNN
+F 2 "Strix:L_0402" H 7250 2700 50  0001 C CNN
 F 3 "" H 7250 2700 50  0001 C CNN
 	1    7250 2700
@@
 F 0 "C26" H 7100 2750 50  0000 C BNN
 F 1 "5p1" H 7100 2650 50  0000 C TNN
-F 2 "Strix:C_0402_1005Metric_Pad0.74x0.62mm_HandSolder" H 7050 2700 50  0001 C CNN
+F 2 "Strix:C_0402" H 7050 2700 50  0001 C CNN
 F 3 "" H 7050 2700 50  0001 C CNN
 	1    7050 2700
@@
 F 0 "C28" V 7804 2858 50  0000 L CNN
 F 1 "6n8" V 7895 2858 50  0000 L CNN
-F 2 "Strix:C_0402_1005Metric_Pad0.74x0.62mm_HandSolder" H 7800 2800 50  0001 C CNN
+F 2 "Strix:C_0402" H 7800 2800 50  0001 C CNN
 F 3 "" H 7800 2800 50  0001 C CNN
 	1    7800 2800
@@
 F 0 "L6" H 8800 2750 50  0000 C BNN
 F 1 "24n" H 8800 2650 50  0000 C TNN
-F 2 "Strix:L_0402_1005Metric_Pad0.77x0.64mm_HandSolder" H 8750 2700 50  0001 C CNN
+F 2 "Strix:L_0402" H 8750 2700 50  0001 C CNN
 F 3 "" H 8750 2700 50  0001 C CNN
 	1    8750 2700
@@
 F 0 "C29" V 8554 2858 50  0000 L CNN
 F 1 "3p3" V 8645 2858 50  0000 L CNN
-F 2 "Strix:C_0402_1005Metric_Pad0.74x0.62mm_HandSolder" H 8550 2800 50  0001 C CNN
+F 2 "Strix:C_0402" H 8550 2800 50  0001 C CNN
 F 3 "" H 8550 2800 50  0001 C CNN
 	1    8550 2800
@@
 F 0 "C30" V 9054 2858 50  0000 L CNN
 F 1 "3p3" V 9145 2858 50  0000 L CNN
-F 2 "Strix:C_0402_1005Metric_Pad0.74x0.62mm_HandSolder" H 9050 2800 50  0001 C CNN
+F 2 "Strix:C_0402" H 9050 2800 50  0001 C CNN
 F 3 "" H 9050 2800 50  0001 C CNN
 	1    9050 2800
@@
 F 0 "L5" H 8200 2750 50  0000 C BNN
 F 1 "12n" H 8200 2650 50  0000 C TNN
-F 2 "Strix:L_0402_1005Metric_Pad0.77x0.64mm_HandSolder" H 8150 2700 50  0001 C CNN
+F 2 "Strix:L_0402" H 8150 2700 50  0001 C CNN
 F 3 "" H 8150 2700 50  0001 C CNN
 	1    8150 2700
@@
 F 0 "L7" H 9400 2750 50  0000 C BNN
 F 1 "12n" H 9400 2650 50  0000 C TNN
-F 2 "Strix:L_0402_1005Metric_Pad0.77x0.64mm_HandSolder" H 9350 2700 50  0001 C CNN
+F 2 "Strix:L_0402" H 9350 2700 50  0001 C CNN
 F 3 "" H 9350 2700 50  0001 C CNN
 	1    9350 2700
@@
 F 0 "C19" V 4450 4950 50  0000 L CNN
 F 1 "100n" V 4350 4950 50  0000 L CNN
-F 2 "Strix:C_0402_1005Metric_Pad0.74x0.62mm_HandSolder" H 4400 4900 50  0001 C CNN
+F 2 "Strix:C_0402" H 4400 4900 50  0001 C CNN
 F 3 "" H 4400 4900 50  0001 C CNN
 	1    4400 4900
@@
 F 0 "C20" V 4450 3750 50  0000 L CNN
 F 1 "1u" V 4550 3750 50  0000 L CNN
-F 2 "Strix:C_0402_1005Metric_Pad0.74x0.62mm_HandSolder" H 4450 3700 50  0001 C CNN
+F 2 "Strix:C_0402" H 4450 3700 50  0001 C CNN
 F 3 "" H 4450 3700 50  0001 C CNN
 	1    4450 3700
@@
 F 0 "C21" V 4700 3750 50  0000 L CNN
 F 1 "2u2" V 4800 3750 50  0000 L CNN
-F 2 "Strix:C_0402_1005Metric_Pad0.74x0.62mm_HandSolder" H 4700 3700 50  0001 C CNN
+F 2 "Strix:C_0402" H 4700 3700 50  0001 C CNN
 F 3 "" H 4700 3700 50  0001 C CNN
 	1    4700 3700
@@
 F 0 "C22" V 5000 3750 50  0000 L CNN
 F 1 "100n" V 5100 3750 50  0000 L CNN
-F 2 "Strix:C_0402_1005Metric_Pad0.74x0.62mm_HandSolder" H 5000 3700 50  0001 C CNN
+F 2 "Strix:C_0402" H 5000 3700 50  0001 C CNN
 F 3 "" H 5000 3700 50  0001 C CNN
 	1    5000 3700
@@
 F 0 "C23" V 5300 3750 50  0000 L CNN
 F 1 "220p" V 5400 3750 50  0000 L CNN
-F 2 "Strix:C_0402_1005Metric_Pad0.74x0.62mm_HandSolder" H 5300 3700 50  0001 C CNN
+F 2 "Strix:C_0402" H 5300 3700 50  0001 C CNN
 F 3 "" H 5300 3700 50  0001 C CNN
 	1    5300 3700
@@
 F 0 "C24" V 5600 3750 50  0000 L CNN
 F 1 "100p" V 5700 3750 50  0000 L CNN
-F 2 "Strix:C_0402_1005Metric_Pad0.74x0.62mm_HandSolder" H 5600 3700 50  0001 C CNN
+F 2 "Strix:C_0402" H 5600 3700 50  0001 C CNN
 F 3 "" H 5600 3700 50  0001 C CNN
 	1    5600 3700
@@
 $EndComp
 $Comp
-L Strix:RF_Shield_Two_Pieces J4
+L Strix:BMI-S-201 J4
 U 1 1 613A4699
 P 8450 5000
+AR Path="/613A4699" Ref="J4"  Part="1"
+AR Path="/611291B2/613A4699" Ref="J4"  Part="1"
 F 0 "J4" H 9180 5064 50  0000 L CNN
 F 1 "BMI-S-201" H 9180 4973 50  0000 L CNN
-F 2 "Strix:Laird_Technologies_BMI-S-201-F_13.66x12.70mm" H 8450 4900 50  0001 C CNN
+F 2 "Strix:BMI-S-201" H 8450 4900 50  0001 C CNN
 F 3 "~" H 8450 4900 50  0001 C CNN
 	1    8450 5000
@@
 F 0 "R11" V 2150 3050 50  0000 L CNN
 F 1 "10k" V 2250 3050 50  0000 L CNN
-F 2 "Strix:R_0402_1005Metric_Pad0.72x0.64mm_HandSolder" H 2150 3000 50  0001 C CNN
+F 2 "Strix:R_0402" H 2150 3000 50  0001 C CNN
 F 3 "" H 2150 3000 50  0001 C CNN
 	1    2150 3000
@@
 F 0 "R4" H 2050 2750 50  0000 C BNN
 F 1 "10k" H 2050 2900 50  0000 C BNN
-F 2 "Strix:R_0402_1005Metric_Pad0.72x0.64mm_HandSolder" H 2000 2850 50  0001 C CNN
+F 2 "Strix:R_0402" H 2000 2850 50  0001 C CNN
 F 3 "" H 2000 2850 50  0001 C CNN
 	1    2000 2850
