File: schematics/altimeter.kicad_sch (KiCad schematic)
At the start: 6 parts, among them U4 TXB0106, U5 MS5611-01BA, U6 ICM-20948

Commit message: Complete revision 1 schematic
Parts:
- removed C17, C18: 100n, Strix:C_0402, symbol Strix:C
- removed U4: TXB0106, symbol Strix:TXB0106
- removed U5: MS5611-01BA, Strix:MS5611-01BA, symbol Strix:MS5611-01BA
- removed U6: ICM-20948, Strix:ICM-20948, symbol Strix:ICM-20948
- added C11, C13: 100p, symbol Strix:C
- added C12, C14: 15p, symbol Strix:C
- added R4, R6, R8, R9: 4k7, symbol Strix:R
- added R5: 200k, symbol Strix:R
- added U3: NVT2006, symbol Strix:NVT2006
- added U4: PCA9306, symbol Strix:PCA9306
- added U5: ICM-20789, Strix:ICM-20789, symbol Strix:ICM-20789
- added U6: MS5611-01BA, Strix:MS5611-01BA, symbol Strix:MS5611-01BA
- R7: value 100k -> 200k; footprint Strix:R_0402 -> (none)
Connections:
- net 1v8: now also R8.1, R9.1, U3.2 (VREFA), U4.2 (VREF1), U5.8 (VDDIO); no longer R7.1
- net 3v3: now also R7.1, C11.2, C13.2, R4.1, R5.1, R6.1, U3.15 (VREFB), U4.7 (VREF2), U5.13 (VDD), U6.1 (VDD)
- net BARO_MISO: now also U6.6 (SDO)
- net BARO_MOSI: now also U6.7 (SDI/SDA)
- net BARO_SCLK: now also U6.8 (SCLK)
- net BARO_~{CS}: now also U6.4 (CSB), U6.5 (CSB)
- net GND: now also C11.1, C12.1, C13.1, C14.1, U3.1 (GND), U4.1 (GND), U5.10 (REGOUT), U5.11 (FSYNC), U5.18 (GND), U5.20 (NC), U6.2 (PS), U6.3 (GND); no longer R7.2
- net IMU_INT: now also U3.10 (B5)
- net IMU_MISO: now also U3.14 (B1)
- net IMU_MOSI: now also U3.13 (B2)
- net IMU_SCLK: now also U3.12 (B3)
- net IMU_~{CS}: now also U3.11 (B4)
- new net: C12.2, R5.2, U3.16 (EN)
- new net: U3.3 (A1), U5.23 (SCL/SCLK)
- new net: U3.4 (A2), U5.9 (SDO/AD0)
- new net: U3.5 (A3), U5.24 (SDA/SDI)
- new net: U3.6 (A4), U5.22 (~{CS})
- new net: U3.7 (A5), U5.12 (INT)
- new net: C14.2, R7.2, U4.8 (EN)
- new net: R9.2, U4.4 (SDA1), U5.6 (PR_DA)
- new net: R8.2, U4.3 (SCL1), U5.7 (PR_CL)
- new net IMU_PR_CL: R4.2, U4.6 (SCL2)
- new net IMU_PR_DA: R6.2, U4.5 (SDA2)
- no-connect marks 4 -> 2
Other:
- note added: "I2C Level Shifter"
- note added: "SPI Level Shifter"
- note removed: "3v3/1v8 Level Shifter"

Commit message: Add oscillators and clean up schematics
Parts:
- C11, C12, C13, C14: footprint (none) -> Strix:C_0402
- R4, R5, R6, R7, R8, R9: footprint (none) -> Strix:R_0402
Connections:
- net IMU_MISO is gone; now on net MISO: U3.14 (B1)
- net IMU_MOSI is gone; now on net MOSI: U3.13 (B2)
- net IMU_SCLK is gone; now on net SCLK: U3.12 (B3)
- net BARO_MISO renamed MISO
- net BARO_MOSI renamed MOSI
- net BARO_SCLK renamed SCLK
Other:
- note added: "7-DoF IMU"
- note added: "Integrated IMU + Barometer"
- note added: "Redundant Barometer"
- note removed: "Barometer"
- note removed: "IMU"
- moved on the sheet: C11, C12, C13, C14, R4, R5, R6, R7, R8, R9, U3, U4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

Commit message: Add missing IC footprints
Parts:
- U3: value NVT2006 -> NVT2006BQ; footprint (none) -> Strix:NVT2006BQ; symbol Strix:NVT2006 -> Strix:NVT2006BQ
- renumbered C11 to C13, C12 to C14, C13 to C15, C14 to C16, R9 to R10, R4 to R5, R5 to R6, R6 to R7, R7 to R8, R8 to R9
Changed lines of the file:
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@@
   (symbol (lib_id "Strix:GND") (at 196.85 105.41 0) (unit 1)
     (in_bom yes) (on_board yes)
-    (property "Reference" "#PWR026" (id 0) (at 193.548 104.394 0)
+    (property "Reference" "#PWR027" (id 0) (at 193.548 104.394 0)
       (effects (font (size 1.27 1.27)) (justify left) hide)
     )
@@
   (symbol (lib_id "Strix:3v3") (at 196.85 82.55 0) (unit 1)
     (in_bom yes) (on_board yes)
-    (property "Reference" "#PWR025" (id 0) (at 196.85 79.756 0)
+    (property "Reference" "#PWR026" (id 0) (at 196.85 79.756 0)
       (effects (font (size 1.27 1.27)) (justify left) hide)
     )
@@
   (symbol (lib_id "Strix:1v8") (at 91.44 46.99 0) (unit 1)
     (in_bom yes) (on_board yes)
-    (property "Reference" "#PWR016" (id 0) (at 91.44 44.196 0)
+    (property "Reference" "#PWR017" (id 0) (at 91.44 44.196 0)
       (effects (font (size 1.27 1.27)) (justify left) hide)
     )
@@
   (symbol (lib_id "Strix:GND") (at 87.63 87.63 0) (mirror y) (unit 1)
     (in_bom yes) (on_board yes)
-    (property "Reference" "#PWR015" (id 0) (at 90.932 86.614 0)
+    (property "Reference" "#PWR016" (id 0) (at 90.932 86.614 0)
       (effects (font (size 1.27 1.27)) (justify left) hide)
     )
@@
   (symbol (lib_id "Strix:1v8") (at 121.92 46.99 0) (unit 1)
     (in_bom yes) (on_board yes)
-    (property "Reference" "#PWR021" (id 0) (at 121.92 44.196 0)
+    (property "Reference" "#PWR022" (id 0) (at 121.92 44.196 0)
       (effects (font (size 1.27 1.27)) (justify left) hide)
     )
@@
   (symbol (lib_id "Strix:3v3") (at 127 46.99 0) (unit 1)
     (in_bom yes) (on_board yes)
-    (property "Reference" "#PWR023" (id 0) (at 127 44.196 0)
+    (property "Reference" "#PWR024" (id 0) (at 127 44.196 0)
       (effects (font (size 1.27 1.27)) (justify left) hide)
     )
@@
   (symbol (lib_id "Strix:GND") (at 124.46 87.63 0) (unit 1)
     (in_bom yes) (on_board yes)
-    (property "Reference" "#PWR022" (id 0) (at 121.158 86.614 0)
+    (property "Reference" "#PWR023" (id 0) (at 121.158 86.614 0)
       (effects (font (size 1.27 1.27)) (justify left) hide)
     )
@@
   (symbol (lib_id "Strix:GND") (at 139.7 87.63 0) (unit 1)
     (in_bom yes) (on_board yes)
-    (property "Reference" "#PWR024" (id 0) (at 136.398 86.614 0)
+    (property "Reference" "#PWR025" (id 0) (at 136.398 86.614 0)
       (effects (font (size 1.27 1.27)) (justify left) hide)
     )
@@
   (symbol (lib_id "Strix:GND") (at 109.22 87.63 0) (unit 1)
     (in_bom yes) (on_board yes)
-    (property "Reference" "#PWR019" (id 0) (at 105.918 86.614 0)
+    (property "Reference" "#PWR020" (id 0) (at 105.918 86.614 0)
       (effects (font (size 1.27 1.27)) (justify left) hide)
     )
@@
   (symbol (lib_id "Strix:C") (at 72.39 82.55 90) (unit 1)
     (in_bom yes) (on_board yes)
-    (property "Reference" "C12" (id 0) (at 71.12 80.01 90)
+    (property "Reference" "C14" (id 0) (at 71.12 80.01 90)
       (effects (font (size 1.27 1.27)) (justify left))
     )
@@
     (pin "2")
   )
-  (symbol (lib_id "Strix:NVT2006") (at 87.63 66.04 0) (mirror y) (unit 1)
-    (in_bom yes) (on_board yes)
-    (property "Reference" "U3" (id 0) (at 92.71 53.34 0)
+  (symbol (lib_id "Strix:NVT2006BQ") (at 87.63 66.04 0) (mirror y) (unit 1)
+    (in_bom yes) (on_board yes)
+    (property "Reference" "U3" (id 0) (at 90.17 82.55 0)
       (effects (font (size 1.27 1.27)) (justify right))
     )
-    (property "Value" "NVT2006" (id 1) (at 92.71 55.88 0)
+    (property "Value" "NVT2006BQ" (id 1) (at 90.17 85.09 0)
       (effects (font (size 1.27 1.27)) (justify right))
     )
-    (property "Footprint" "" (id 2) (at 87.63 65.405 0)
+    (property "Footprint" "Strix:NVT2006BQ" (id 2) (at 87.63 65.405 0)
       (effects (font (size 1.27 1.27)) hide)
     )
@@
   (symbol (lib_id "Strix:C") (at 93.98 132.08 90) (unit 1)
     (in_bom yes) (on_board yes)
-    (property "Reference" "C14" (id 0) (at 92.71 129.54 90)
+    (property "Reference" "C16" (id 0) (at 92.71 129.54 90)
       (effects (font (size 1.27 1.27)) (justify left))
     )
@@
   (symbol (lib_id "Strix:R") (at 127 114.3 270) (unit 1)
     (in_bom yes) (on_board yes)
-    (property "Reference" "R9" (id 0) (at 128.27 114.3 90)
+    (property "Reference" "R10" (id 0) (at 128.27 114.3 90)
       (effects (font (size 1.27 1.27)) (justify left))
     )
@@
   (symbol (lib_id "Strix:R") (at 124.46 114.3 90) (mirror x) (unit 1)
     (in_bom yes) (on_board yes)
-    (property "Reference" "R8" (id 0) (at 123.19 114.3 90)
+    (property "Reference" "R9" (id 0) (at 123.19 114.3 90)
       (effects (font (size 1.27 1.27)) (justify left))
     )
@@
   (symbol (lib_id "Strix:GND") (at 209.55 105.41 0) (unit 1)
     (in_bom yes) (on_board yes)
-    (property "Reference" "#PWR027" (id 0) (at 206.248 104.394 0)
+    (property "Reference" "#PWR028" (id 0) (at 206.248 104.394 0)
       (effects (font (size 1.27 1.27)) (justify left) hide)
     )
@@
   (symbol (lib_id "Strix:C") (at 62.23 82.55 90) (unit 1)
     (in_bom yes) (on_board yes)
-    (property "Reference" "C11" (id 0) (at 60.96 80.01 90)
+    (property "Reference" "C13" (id 0) (at 60.96 80.01 90)
       (effects (font (size 1.27 1.27)) (justify left))
     )
@@
   (symbol (lib_id "Strix:1v8") (at 109.22 104.14 0) (unit 1)
     (in_bom yes) (on_board yes)
-    (property "Reference" "#PWR020" (id 0) (at 109.22 101.346 0)
+    (property "Reference" "#PWR021" (id 0) (at 109.22 101.346 0)
       (effects (font (size 1.27 1.27)) (justify left) hide)
     )
@@
   (symbol (lib_id "Strix:3v3") (at 83.82 46.99 0) (unit 1)
     (in_bom yes) (on_board yes)
-    (property "Reference" "#PWR014" (id 0) (at 83.82 44.196 0)
+    (property "Reference" "#PWR015" (id 0) (at 83.82 44.196 0)
       (effects (font (size 1.27 1.27)) (justify left) hide)
     )
@@
   (symbol (lib_id "Strix:GND") (at 106.68 139.7 0) (mirror y) (unit 1)
     (in_bom yes) (on_board yes)
-    (property "Reference" "#PWR018" (id 0) (at 109.982 138.684 0)
+    (property "Reference" "#PWR019" (id 0) (at 109.982 138.684 0)
       (effects (font (size 1.27 1.27)) (justify left) hide)
     )
@@
   (symbol (lib_id "Strix:R") (at 71.12 114.3 90) (mirror x) (unit 1)
     (in_bom yes) (on_board yes)
-    (property "Reference" "R4" (id 0) (at 69.85 114.3 90)
+    (property "Reference" "R5" (id 0) (at 69.85 114.3 90)
       (effects (font (size 1.27 1.27)) (justify left))
     )
@@
   (symbol (lib_id "Strix:R") (at 72.39 72.39 90) (mirror x) (unit 1)
     (in_bom yes) (on_board yes)
-    (property "Reference" "R5" (id 0) (at 71.12 72.39 90)
+    (property "Reference" "R6" (id 0) (at 71.12 72.39 90)
       (effects (font (size 1.27 1.27)) (justify left))
     )
@@
   (symbol (lib_id "Strix:R") (at 73.66 114.3 270) (unit 1)
     (in_bom yes) (on_board yes)
-    (property "Reference" "R6" (id 0) (at 74.93 114.3 90)
+    (property "Reference" "R7" (id 0) (at 74.93 114.3 90)
       (effects (font (size 1.27 1.27)) (justify left))
     )
@@
   (symbol (lib_id "Strix:3v3") (at 104.14 104.14 0) (unit 1)
     (in_bom yes) (on_board yes)
-    (property "Reference" "#PWR017" (id 0) (at 104.14 101.346 0)
+    (property "Reference" "#PWR018" (id 0) (at 104.14 101.346 0)
       (effects (font (size 1.27 1.27)) (justify left) hide)
     )
@@
   (symbol (lib_id "Strix:R") (at 93.98 114.3 90) (mirror x) (unit 1)
     (in_bom yes) (on_board yes)
-    (property "Reference" "R7" (id 0) (at 92.71 114.3 90)
+    (property "Reference" "R8" (id 0) (at 92.71 114.3 90)
       (effects (font (size 1.27 1.27)) (justify left))
     )
@@
   (symbol (lib_id "Strix:C") (at 83.82 132.08 90) (unit 1)
     (in_bom yes) (on_board yes)
-    (property "Reference" "C13" (id 0) (at 82.55 129.54 90)
-      (effects (font (size 1.27 1.27)) (justify left))
-    )
+    (property "Reference" "C15" (id 0) (at 82.55 129.54 90)
+      (effects (font (size 1.27 1.27)) (justify left))
+    )

Commit message: Fix outdated footprint references in symbol lib
Parts:
- U4: footprint (none) -> Strix:PCA9306
Changed lines of the file:
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@@
       (effects (font (size 1.27 1.27)) (justify right))
     )
-    (property "Footprint" "" (id 2) (at 116.84 113.03 0)
+    (property "Footprint" "Strix:PCA9306" (id 2) (at 116.84 113.03 0)
       (effects (font (size 1.27 1.27)) hide)
     )
