File: schematics/flight-computer/psu.kicad_sch (KiCad schematic)
At the start: 18 parts, among them U401 MAX604, U402 BQ29200, U403 MAX604

Commit message: Update passive order codes to 0402
Parts:
- C403, C404, C405: Farnell 1759166 -> 2496771
- C406: Farnell 2346946 -> 2627379
- R401, R403, R405: Farnell 2447552 -> 2447095
- R402, R404: Farnell 2694996 -> 2331465
Changed lines of the file:
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@@
       (effects (font (size 1.27 1.27)) hide)
     )
-    (property "Farnell" "1759166" (id 4) (at 114.3 62.23 0)
+    (property "Farnell" "2496771" (id 4) (at 114.3 62.23 0)
       (effects (font (size 1.27 1.27)) hide)
     )
@@
       (effects (font (size 1.27 1.27)) hide)
     )
-    (property "Farnell" "1759166" (id 4) (at 62.23 67.31 0)
+    (property "Farnell" "2496771" (id 4) (at 62.23 67.31 0)
       (effects (font (size 1.27 1.27)) hide)
     )
@@
       (effects (font (size 1.27 1.27)) hide)
     )
-    (property "Farnell" "1759166" (id 4) (at 62.23 59.69 0)
+    (property "Farnell" "2496771" (id 4) (at 62.23 59.69 0)
       (effects (font (size 1.27 1.27)) hide)
     )
@@
       (effects (font (size 1.27 1.27)) hide)
     )
-    (property "Farnell" "2346946" (id 4) (at 74.93 73.66 0)
+    (property "Farnell" "2627379" (id 4) (at 74.93 73.66 0)
       (effects (font (size 1.27 1.27)) hide)
     )
@@
       (effects (font (size 1.27 1.27)) hide)
     )
-    (property "Farnell" "2447552" (id 4) (at 50.8 72.39 0)
+    (property "Farnell" "2447095" (id 4) (at 50.8 72.39 0)
       (effects (font (size 1.27 1.27)) hide)
     )
@@
       (effects (font (size 1.27 1.27)) hide)
     )
-    (property "Farnell" "2447552" (id 4) (at 46.99 64.77 0)
+    (property "Farnell" "2447095" (id 4) (at 46.99 64.77 0)
       (effects (font (size 1.27 1.27)) hide)
     )
@@
       (effects (font (size 1.27 1.27)) hide)
     )
-    (property "Farnell" "2447552" (id 4) (at 114.3 48.26 0)
+    (property "Farnell" "2447095" (id 4) (at 114.3 48.26 0)
       (effects (font (size 1.27 1.27)) hide)
     )
@@
       (effects (font (size 1.27 1.27)) hide)
     )
-    (property "Farnell" "2694996" (id 4) (at 54.61 64.77 0)
+    (property "Farnell" "2331465" (id 4) (at 54.61 64.77 0)
       (effects (font (size 1.27 1.27)) hide)
     )
@@
       (effects (font (size 1.27 1.27)) hide)
     )
-    (property "Farnell" "2694996" (id 4) (at 50.8 57.15 0)
-      (effects (font (size 1.27 1.27)) hide)
-    )
+    (property "Farnell" "2331465" (id 4) (at 50.8 57.15 0)
+      (effects (font (size 1.27 1.27)) hide)
+    )
